File: Kicad/Projects/PCB Design Mastery Course/DF-ESC/Design/rev01/rev01_1/DF_ESC_rev01.1/MOSFET_DRIVER.kicad_sch (KiCad schematic)
At the start: 0 parts

Commit message: Update 6
Building MOS-FET Driver Schematic
Parts:
- added C301: 120p, symbol Device:C
- added C302: 6n8, symbol Device:C
- added C303, C304, C305, C306, C307, C308: 2u2, symbol Device:C
- added C309, C310, C311, C312, C313, C314, C315, C316, C317: 10u, symbol Device:C
- added C318: 100n, symbol Device:C
- added C319: 100u, symbol Device:C_Polarized
- added C320, C321, C322: 220n, symbol Device:C
- added D301: B220, Diode_SMD:D_SMB, symbol Diode:B220
- added D302: BAT60A, Diode_SMD:D_SOD-323, symbol Diode:BAT60A
- added L301: 22u, symbol Device:L
- added R301: 205k, symbol Device:R
- added R302: 16k2, symbol Device:R
- added R303, R309, R311: 39k, symbol Device:R
- added R304, R310, R312: 2k2, symbol Device:R
- added R305, R306: 10k, symbol Device:R
- added R307: 3k3, symbol Device:R
- added R308: 1M, symbol Device:R
- added U301: DRV8302DCAR, DCA56_6P35X3P61, symbol DRV8302:DRV8302DCAR
Connections:
- new net: R301.2, U301.1 (RT_CLK)
- new net: C305.1, C306.1, U301.13 (GVDD)
- new net: C302.2, R302.1
- new net: C301.1, R302.2, U301.2 (COMP)
- new net: C307.1, U301.14 (CP1)
- new net: C307.2, U301.15 (CP2)
- new net: C308.1, U301.27 (AVDD)
- new net: R308.1, U301.49 (BIAS)
- new net: R305.2, U301.7 (DTC)
- new net +3V3: U301.24 (REF), U301.9 (M_OC)
- new net +5V: D302.1 (K)
- new net +5V_VDD: C319.1, D302.2 (A), L301.2, R306.1
- new net +VDC: C309.1, C310.1, C311.1, C312.1, C313.1, C314.1, C315.1, C316.1, C317.1, U301.29 (PVDD1), U301.53 (PVDD2), U301.54 (PVDD2)
- new net BR_SO1: U301.25 (SO1)
- new net BR_SO2: U301.26 (SO2)
- new net BST_A: C320.1, U301.48 (BST_A)
- new net BST_B: C321.1, U301.43 (BST_B)
- new net BST_BK: C318.1, U301.52 (BST_BK)
- new net BST_C: C322.1, U301.38 (BST_C)
- new net DC_CAL: U301.12 (DC_CAL)
- new net DVDD: C303.1, C304.1, U301.11 (OC_ADJ), U301.23 (DVDD)
- new net EN_GATE: U301.16 (EN_GATE)
- new net FAULT: U301.6 (*FAULT)
- new net GH_A: U301.47 (GH_A)
- new net GH_B: U301.42 (GH_B)
- new net GH_C: U301.37 (GH_C)
- new net GL_A: U301.45 (GL_A)
- new net GL_B: U301.40 (GL_B)
- new net GL_C: U301.35 (GL_C)
- new net GND: C301.2, C302.1, C303.2, C304.2, C305.2, C306.2, C308.2, C309.2, C310.2, C311.2, C312.2, C313.2, C314.2, C315.2, C316.2, C317.2, C319.2, D301.2 (A), R301.1, R304.1, R305.1, R307.2, R308.2, R310.1, R312.1, U301.10 (GAIN), U301.28 (AGND), U301.57 (EPAD), U301.8 (M_PWM)
- new net H1: U301.17 (INH_A)
- new net H2: U301.19 (INH_B)
- new net H3: U301.21 (INH_C)
- new net L1: U301.18 (INL_A)
- new net L2: U301.20 (INL_B)
- new net L3: U301.22 (INL_C)
- new net PH: C318.2, D301.1 (K), L301.1, U301.50 (PH), U301.51 (PH)
- new net SENS1: R303.2, R304.2
- new net SENS2: R309.2, R310.2
- new net SENS3: R311.2, R312.2
- new net SH_A: C320.2, U301.46 (SH_A)
- new net SH_B: C321.2, U301.41 (SH_B)
- new net SH_C: C322.2, U301.36 (SH_C)
- new net SL_A: R303.1, U301.44 (SL_A)
- new net SL_B: R309.1, U301.39 (SL_B)
- new net SL_C: R311.1, U301.34 (SL_C)
- new net SN1: U301.33 (SN1)
- new net SN2: U301.31 (SN2)
- new net SP1: U301.32 (SP1)
- new net SP2: U301.30 (SP2)
- new net VSENSE: R306.2, R307.1, U301.3 (VSENSE)
- no-connect marks 0 -> 4
Other:
- note added: "10uF DECOUPLING CAPACITORS PLACE AS CLOSE AS POSSIBLE TO THE IC PVDD2 PINS"
- note added: "BULK CAPACITANCE KEEP AS CLOSE AS POSSIBLE TO THE IC AND TO THE DRIVER INPUT LOOP"
- note added: "INPUT PORTS"
- note added: "OUTPUT PORTS"
- note added: "TYPICAL APPLICATION SCHEMATIC"

Commit message: Update 7
Completed MOSFET_DRIVER Schematic
Parts:
- removed C319: 100u, symbol Device:C_Polarized
- removed D301: B220, Diode_SMD:D_SMB, symbol Diode:B220
- added C319, C323, C324: 10u, symbol Device:C
- added D301: PMEG6020AELR, Diode_SMD:Nexperia_CFP3_SOD-123W, symbol Diode:PMEG6020AELR
- C302: value 6n8 -> 10n
- C307: value 2u2 -> 22n
- C309, C310, C311: value 10u -> 100n
- C312, C313, C314, C315, C316, C317: value 10u -> 1u
- R302: value 16k2 -> 16k
- R306: value 10k -> 18k
- U301: footprint DCA56_6P35X3P61 -> Motor_Drivers:HTSSOP-56_L14.0-W6.1-P0.50-LS8.1-BL-EP
Connections:
- net GND: now also C319.2, C323.2, C324.2, D301.2 (A)
- net PH: now also D301.1 (K)
- net +5V_VDD renamed +5V_DRV
- net +5V_DRV: now also C319.1, C323.1, C324.1
- net GH_A renamed MH_1
- net GH_B renamed MH_2
- net GH_C renamed MH_3
- net GL_A renamed M_L1
- net GL_B renamed M_L2
- net GL_C renamed M_L3
- net SH_A renamed H1_VS
- net H1_VS: now also R311.1
- net SH_B renamed H2_VS
- net H2_VS: now also R309.1
- net SH_C renamed H3_VS
- net H3_VS: now also R303.1
- net SL_A renamed H1_LOW
- net H1_LOW: no longer R303.1
- net SL_B renamed H2_LOW
- net H2_LOW: no longer R309.1
- net SL_C renamed H3_LOW
- net H3_LOW: no longer R311.1
Other:
- note added: "BOOTSTRAP CAPACITORS"
- note added: "Hx_VS"
- note added: "KEEP AWAY FROM NOISY TRACKS AND COMPONENTS"
- note added: "MCU SENSING FEEDBACK FOR EACH PHASE"
- note added: "PHASE 1"
- note added: "PHASE 2"
- note added: "PHASE 3"
- note added: "SENSE 1 - PHASE 3"
- note added: "SENSE 2 - PHASE 1"
- note added: "[03] - ${SHEETNAME}"
- moved on the sheet: C301, C302, C303, C304, C305, C306, C307, C308, C309, C310, C311, C312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
